File: DP-Switching.kicad_sch (KiCad schematic)
At the start: 22 parts, among them J2 E9320-001-01, J3 E9320-001-01, J4 E9320-001-01, J5 E9320-001-01, U1 TS3DV642A0RUAR, U2 TS3DV642A0RUAR

Commit message: Add titles, dates, and company
Other:
- title: (none) -> DisplayPort Switching
Changed lines of the file:
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@@
 	(paper "USLetter")
 	(title_block
+		(title "DisplayPort Switching")
+		(date "21-Feb-2025")
 		(rev "1")
 		(company "rieberger.ca")
