File: Enable-Counter.kicad_sch (KiCad schematic)
At the start: 16 parts, among them SW1 SW_Push, U3 SN74LVC112AD, U4 74LVC1G04, U5 74LVC1G04, U6 TLC555xD, U7 74LVC1G02, U8 74LVC1G08

Commit message: Add titles, dates, and company
Other:
- company: (none) -> rieberger.ca
- title: (none) -> Enable Counter
Changed lines of the file:
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@@
 	(generator_version "9.0")
 	(paper "USLetter")
+	(title_block
+		(title "Enable Counter")
+		(date "24-Feb-2025")
+		(rev "1")
+		(company "rieberger.ca")
+	)
 	(text "Debounce circuit"
 		(exclude_from_sim no)
