File: USB-Switching.kicad_sch (KiCad schematic)
At the start: 4 parts, among them J10 USB_A_Stacked, J7 USB_A_Stacked, J8 USB_A_Stacked, J9 USB_A_Stacked

Commit message: Add titles, dates, and company
Other:
- company: (none) -> rieberger.ca
- title: (none) -> USB Switching
Changed lines of the file:
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@@
 	(generator_version "9.0")
 	(paper "USLetter")
+	(title_block
+		(title "USB Switching")
+		(date "23-Mar-2025")
+		(rev "1")
+		(company "rieberger.ca")
+	)
 	(symbol
 		(lib_id "Connector:USB_A_Stacked")
